Commit message: 4-wheel implementation
Added 2 additional joints and modified original format

File: urdf/kangaroo_diff_drive.xacro (robot description, xacro)
@@ -3,49 +3,44 @@
   <!-- Constants for robot dimensions -->
   <xacro:property name="PI" value="3.1415926535897931"/>
+  <xacro:property name = "chassis_width" value = "0.3"/>
+  <xacro:property name = "axle_width" value = "0.46"/>
+  <xacro:property name = "length" value = "0.6"/>
+  <xacro:property name = "wheel_t" value = "0.03"/>
+  <xacro:property name = "wheel_r" value = "0.2"/>
   <!-- Base Link -->
-  <link name="base_link"/>
-  <link name="left_wheel">
-    <collision name="collision">
-      <origin xyz="0 0.0 0" rpy="0 1.5707 1.5707"/>
-      <geometry>
-         <cylinder  length="0.03" radius="0.045"/>
-      </geometry>
-    </collision>
-    <visual name="visual">
-      <origin xyz="0 0.0 0" rpy="0 1.5707 1.5707"/>
-      <geometry>
-        <cylinder  length="0.03" radius="0.045"/>
-      </geometry>
-      <material name="black"/>
-    </visual>
-  </link>
-  <joint type="revolute" name="motor_2_joint">
-    <origin xyz="0 0.15 0" rpy="0 0 0"/>
-    <child link="left_wheel">left_wheel</child>
-    <parent link="base_link">base_link</parent>
-    <axis xyz="0 1 0"/>
-    <limit effort="100" velocity="100.0"  lower="-5000" upper="5000" />
-  </joint>
-  <link name="right_wheel">
-    <collision name="collision">
-      <origin xyz="0 0.0 0" rpy="0 1.5707 1.5707"/>
-      <geometry>
-         <cylinder  length="0.03" radius="0.045"/>
-      </geometry>
-    </collision>
-    <visual name="visual">
-      <origin xyz="0 0.0 0" rpy="0 1.5707 1.5707"/>
-      <geometry>
-        <cylinder  length="0.03" radius="0.045"/>
-      </geometry>
-      <material name="black"/>
-    </visual>
-  </link>
-  <joint type="revolute" name="motor_1_joint">
-    <origin xyz="0 -0.15 0" rpy="0 0 0"/>
-    <child link="right_wheel">right_wheel</child>
-    <parent link="base_link">base_link</parent>
-    <axis xyz="0 1 0"/>
-    <limit effort="100" velocity="100.0"  lower="-5000" upper="5000" />
-  </joint>
+  <link name="base_link">
+     <visual>
+          <geometry>
+               <box size="${length} ${chassis_width} 0.01"/>
+          </geometry>
+     </visual>
+   </link>
+   <xacro:macro name = "wheel" params = "prefix reflect_lr reflect_fr">
+        <link name = "${prefix}_wheel">
+             <collision name="collision">
+               <origin xyz="0 0.0 0" rpy="0 1.5707 1.5707"/>
+               <geometry>
+                  <cylinder  length="${wheel_t}" radius="${wheel_r}"/>
+               </geometry>
+             </collision>
+             <visual name="visual">
+               <origin xyz="0 0.0 0" rpy="0 1.5707 1.5707"/>
+               <geometry>
+                 <cylinder  length="${wheel_t}" radius="${wheel_r}"/>
+               </geometry>
+               <material name="black"/>
+             </visual>
+           </link>
+           <joint type="continuous" name="${prefix}_motor_joint">
+             <origin xyz="${reflect_fr*length/2} ${reflect_lr*axle_width/2} 0" rpy="0 0 0"/>
+             <child link="${prefix}_wheel"/>
+             <parent link="base_link"/>
+             <axis xyz="0 1 0"/>
+             <limit effort="100" velocity="100.0" />
+           </joint>
+      </xacro:macro>
+      <xacro:wheel prefix = "front_left" reflect_lr = "-1" reflect_fr = "1"/>
+      <xacro:wheel prefix = "front_right" reflect_lr = "1" reflect_fr = "1"/>
+      <xacro:wheel prefix = "rear_left" reflect_lr = "-1" reflect_fr = "-1"/>
+      <xacro:wheel prefix = "rear_right" reflect_lr = "1" reflect_fr = "-1"/>
 </robot>
